File: C64PALClockGen.kicad_sch (KiCad schematic)
At the start: 21 parts, among them J1 Conn_01x08_Pin, J2 Conn_01x08_Pin, U1 74AHCT1G125, U2 LDL1117S33, U3 74AHCT1G125, Y1 5V49EE902

Commit message: Finalized v2 dual layer
Parts:
- removed H1, H2: MountingHole, MountingHole:ToolingHole_1.152mm, symbol Mechanical:MountingHole
- added TP1: CLKIN, TestPoint:TestPoint_Pad_D1.0mm, symbol Connector:TestPoint
Connections:
- net XCLKIN: now reaches Y1.5 (CLKIN)
- net XCLKIN: now also TP1.1
- no-connect marks 22 -> 21
Changed lines of the file:
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@@
 (kicad_sch
-	(version 20260326)
+	(version 20260306)
 	(generator "eeschema")
-	(generator_version "10.99")
+	(generator_version "10.0")
 	(paper "A4")
 	(title_block
@@
 	)
 	(no_connect
-		(at 101.6 120.65)
-	)
-	(no_connect
 		(at 129.54 130.81)
 	)
@@
 	(wire
 		(pts
+			(xy 97.79 119.38) (xy 97.79 120.65)
+		)
+		(stroke
+			(width 0)
+			(type default)
+		)
+	)
+	(wire
+		(pts
 			(xy 50.8 55.88) (xy 59.69 55.88)
 		)
@@
 	(wire
 		(pts
+			(xy 97.79 120.65) (xy 101.6 120.65)
+		)
+		(stroke
+			(width 0)
+			(type default)
+		)
+	)
+	(wire
+		(pts
 			(xy 59.69 105.41) (xy 59.69 113.03)
 		)
@@
 		)
 	)
+	(label "XCLKIN"
+		(at 97.79 120.65 0)
+		(effects
+			(font
+				(size 1.27 1.27)
+			)
+			(justify left bottom)
+		)
+	)
 	(label "SDA"
 		(at 92.71 133.35 0)
@@
 	)
 	(symbol
-		(lib_id "Mechanical:MountingHole")
-		(at 21.59 25.4 0)
-		(unit 1)
-		(body_style 1)
-		(exclude_from_sim no)
-		(in_bom no)
-		(on_board yes)
-		(in_pos_files yes)
-		(dnp no)
-		(fields_autoplaced yes)
-		(property "Reference" "H2"
-			(at 24.13 24.1299 0)
-			(show_name no)
-			(do_not_autoplace no)
-			(effects
-				(font
-					(size 1.27 1.27)
-				)
-				(justify left)
-			)
-		)
-		(property "Value" "MountingHole"
-			(at 24.13 26.6699 0)
-			(show_name no)
-			(do_not_autoplace no)
-			(effects
-				(font
-					(size 1.27 1.27)
-				)
-				(justify left)
-			)
-		)
-		(property "Footprint" "MountingHole:ToolingHole_1.152mm"
-			(at 21.59 25.4 0)
-			(hide yes)
-			(show_name no)
-			(do_not_autoplace no)
-			(effects
-				(font
-					(size 1.27 1.27)
-				)
-			)
-		)
-		(property "Datasheet" ""
-			(at 21.59 25.4 0)
-			(hide yes)
-			(show_name no)
-			(do_not_autoplace no)
-			(effects
-				(font
-					(size 1.27 1.27)
-				)
-			)
-		)
-		(property "Description" "Mounting Hole without connection"
-			(at 21.59 25.4 0)
-			(hide yes)
-			(show_name no)
-			(do_not_autoplace no)
-			(effects
-				(font
-					(size 1.27 1.27)
-				)
-			)
-		)
-		(instances
-			(project "C64PALClockGen"
-				(path "/243a460f-1cbe-4d46-a885-532f2a587172"
-					(reference "H2")
-					(unit 1)
-				)
-			)
-		)
-	)
-	(symbol
 		(lib_id "power:GND")
 		(at 173.99 148.59 0)
@@
 	)
 	(symbol
-		(lib_id "Mechanical:MountingHole")
-		(at 21.59 19.05 0)
-		(unit 1)
-		(body_style 1)
-		(exclude_from_sim no)
-		(in_bom no)
-		(on_board yes)
-		(in_pos_files yes)
-		(dnp no)
-		(fields_autoplaced yes)
-		(property "Reference" "H1"
-			(at 24.13 17.7799 0)
-			(show_name no)
-			(do_not_autoplace no)
-			(effects
-				(font
-					(size 1.27 1.27)
-				)
-				(justify left)
-			)
-		)
-		(property "Value" "MountingHole"
-			(at 24.13 20.3199 0)
-			(show_name no)
-			(do_not_autoplace no)
-			(effects
-				(font
-					(size 1.27 1.27)
-				)
-				(justify left)
-			)
-		)
-		(property "Footprint" "MountingHole:ToolingHole_1.152mm"
-			(at 21.59 19.05 0)
-			(hide yes)
-			(show_name no)
-			(do_not_autoplace no)
-			(effects
-				(font
-					(size 1.27 1.27)
-				)
-			)
-		)
-		(property "Datasheet" ""
-			(at 21.59 19.05 0)
-			(hide yes)
-			(show_name no)
-			(do_not_autoplace no)
-			(effects
-				(font
-					(size 1.27 1.27)
-				)
-			)
-		)
-		(property "Description" "Mounting Hole without connection"
-			(at 21.59 19.05 0)
-			(hide yes)
-			(show_name no)
-			(do_not_autoplace no)
-			(effects
-				(font
-					(size 1.27 1.27)
-				)
-			)
-		)
-		(instances
-			(project "C64PALClockGen"
-				(path "/243a460f-1cbe-4d46-a885-532f2a587172"
-					(reference "H1")
-					(unit 1)
-				)
-			)
-		)
-	)
-	(symbol
 		(lib_id "power:PWR_FLAG")
 		(at 119.38 53.34 0)
@@
 					(unit 1)
 				)
+			)
+		)
+	)
+	(symbol
+		(lib_id "Connector:TestPoint")
+		(at 97.79 119.38 0)
+		(unit 1)
+		(body_style 1)
+		(exclude_from_sim no)
+		(in_bom yes)
+		(on_board yes)
+		(in_pos_files yes)
+		(dnp no)
+		(fields_autoplaced yes)
+		(property "Reference" "TP1"
+			(at 100.33 114.8079 0)
+			(show_name no)
+			(do_not_autoplace no)
+			(effects
+				(font
+					(size 1.27 1.27)
+				)
+				(justify left)
+			)
+		)
+		(property "Value" "CLKIN"
+			(at 100.33 117.3479 0)
+			(show_name no)
+			(do_not_autoplace no)
+			(effects
+				(font
+					(size 1.27 1.27)
+				)
+				(justify left)
+			)
+		)
+		(property "Footprint" "TestPoint:TestPoint_Pad_D1.0mm"
+			(at 102.87 119.38 0)
+			(hide yes)
+			(show_name no)
+			(do_not_autoplace no)
+			(effects
+				(font
+					(size 1.27 1.27)
+				)
+			)
+		)
+		(property "Datasheet" ""
+			(at 102.87 119.38 0)
+			(hide yes)
+			(show_name no)
+			(do_not_autoplace no)
+			(effects
+				(font
+					(size 1.27 1.27)
+				)
+			)
+		)
+		(property "Description" "test point"
+			(at 97.79 119.38 0)
+			(hide yes)
+			(show_name no)
+			(do_not_autoplace no)
+			(effects
+				(font
+					(size 1.27 1.27)
+				)
+			)
+		)
+		(pin "1"
+		)
+		(instances
+			(project "C64PALClockGen"
+				(path "/243a460f-1cbe-4d46-a885-532f2a587172"
+					(reference "TP1")
+					(unit 1)
+				)

Commit message: C64 Clock Generator Rev.B
Parts:
- added C10, C11: 100n, Resistor_SMD:R_0603_1608Metric_Pad0.98x0.95mm_HandSolder, symbol Device:C
- added TP2: SDA, TestPoint:TestPoint_Pad_D1.0mm, symbol Connector:TestPoint
- added TP3: SCL, TestPoint:TestPoint_Pad_D1.0mm, symbol Connector:TestPoint
- renumbered C8 to C5, C5 to C6, C10 to C7, C9 to C8, C7 to C9, U2 to U1, U3 to U2, U1 to U3
Connections:
- net +3V3: now also Y1.25 (VDDO3), Y1.9 (VDDO1), C10.1, C11.1
- net GND: now also C10.2, C11.2
- net SCL: now also TP3.1
- net SDA: now also TP2.1
- no-connect marks 21 -> 7
Other:
- note added: "Application Note: DOTCLK: 7.875 MHz COLCLK: 17.734475 MHz"
- note added: "C64 U20"
- note added: "Layout Note: Place decoupling caps close to respective supply pins of Y1"
- note added: "Level Shifter"
- note added: "PLL"
- note added: "Power"
- title: C64 Clock Gen -> C64 Clock Generator
- moved on the sheet: C3, C4, C5, C6, C7, C8, C9, J1, J2, R1, R2, R3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
